Commit message: tried something

File: install/arm_robot/share/arm_robot/arm.urdf.xacro (robot description, xacro)
@@ -6,19 +6,20 @@
 -->
 <robot xmlns:xacro="http://www.ros.org/wiki/xacro" name="arm_robot">
-  <xacro:arg name="prefix" default=""/>
-  <!-- Import RRBot macro -->
+  <xacro:arg name="prefix" default=""/> <!-- By changing the default value you can add a prefix to each link and joint-->
+  <!-- Import arm macro -->
   <xacro:include filename="$(find arm_robot)/arm_description.urdf.xacro" />
   <!-- Import Rviz colors -->
   <!-- <xacro:include filename="$(find 3DOFs_arm)/description/arm.materials.xacro" /> -->
   <!-- Import RRBot ros2_control description -->
-  <xacro:include filename="$(find arm_robot)/arm.ros2_control.xacro" />
+  <!-- <xacro:include filename="$(find arm_robot)/arm.ros2_control.xacro" /> -->
   <!-- Used for fixing robot -->
-  <link name="world"/>
-  <gazebo reference="world">
+  <link name="world">
+  </link>
+  <!-- <gazebo reference="world">
     <static>true</static>
-  </gazebo>
+  </gazebo> -->
   <xacro:arm parent="world" prefix="$(arg prefix)">
     <origin xyz="0 0 0" rpy="0 0 0" />
   </xacro:arm>
-  <xacro:arm_ros2_control name="arm" prefix="$(arg prefix)" />
+  <!-- <xacro:arm_ros2_control name="arm" prefix="$(arg prefix)" /> -->
 </robot>

File: install/arm_robot/share/arm_robot/arm_description.urdf.xacro (robot description, xacro)
@@ -6,13 +6,13 @@
         <xacro:property name="mass" value="1" /> <!-- arbitrary value for mass -->
         <xacro:property name="width" value="0.1" /> <!-- Square dimensions (widthxwidth) of beams -->
-        <xacro:property name="height1" value="2" /> <!-- Link 1 -->
+        <xacro:property name="height1" value="1" /> <!-- Link 1 -->
         <xacro:property name="height2" value="1" /> <!-- Link 2 -->
         <xacro:property name="offset" value="0.05" />
-        <joint name="${prefix}base" type="fixed">
-            <xacro:insert_block name="origin" />
-            <parent link="${parent}" />
-            <child link="${prefix}arm1"/>
+        <joint name="${prefix}base_joint" type="fixed">
+            <xacro:insert_block name="origin"/>
+            <parent link="${parent}"/>
+            <child link="${prefix}base_link"/>
         </joint>
-        <link name="${prefix}arm1">
+        <link name="${prefix}base_link">
             <collision>
                 <origin xyz="0 0 ${height1 / 2}" rpy="0 0 0"/>
@@ -28,20 +28,20 @@
             </visual>
             <interial>
-                <origin xyz="0 0 ${height1 / 2}"/>
+                <origin xyz="0 0 ${height1 / 2}" rpy="0 0 0"/>
                 <mass value="${mass}" />
                 <inertia ixx="${mass / 12 * (width*width + height1*height1)}" ixy="0.0" ixz="0.0" iyy="{mass / 12 * (width*width + height1*height1)}" iyz="0.0" izz="{mass / 12 * 2*width*width}"/>
             </interial>
         </link>
-        <joint name="${prefix}joint1" type="revolute">
-            <parent link="${prefix}arm1"/>
-            <child link="${prefix}arm2"/>
-            <origin xyz="0 ${width} ${height1 / 2 - offset}"/>
+        <!-- <joint name="${prefix}joint1" type="revolute">
+            <parent link="${prefix}base_link"/>
+            <child link="${prefix}arm1_link"/>
+            <origin xyz="0 ${width} ${height1 - offset}" rpy="0 0 0"/>
             <axis xyz="0.0 1.0 0.0"/>
             <limit lower="${-pi}" upper="${pi}" effort="10" velocity="10"/>
             <dynamics damping="0.7"/>
         </joint>
-        <link name="${prefix}arm2">
+        <link name="${prefix}arm1_link">
             <collision>
-                <origin xyz="0 ${width} ${height2 / 2 - offset}" rpy="0 0 0"/>
+                <origin xyz="0 0 ${height2 / 2}" rpy="0 0 0"/>
                 <geometry>
                     <box size="${width} ${width} ${height2}"/>
@@ -49,5 +49,5 @@
             </collision>
             <visual>
-                <origin xyz="0 ${width} ${height2 / 2 - offset}" rpy="0 ${pi} 0"/>
+                <origin xyz="0 0 ${height2 / 2}" rpy="0 0 0"/>
                 <geometry>
                     <box size="${width} ${width} ${height2}"/>
@@ -55,9 +55,9 @@
             </visual>
             <interial>
-                <origin xyz="0 0 ${height2 / 2 - offset}"/>
+                <origin xyz="0 0 ${height2 / 2}" rpy="0 0 0"/>
                 <mass value="${mass}" />
                 <inertia ixx="${mass / 12 * (width*width + height2*height2)}" ixy="0.0" ixz="0.0" iyy="{mass / 12 * (width*width + height2*height2)}" iyz="0.0" izz="{mass / 12 * 2*width*width}"/>
             </interial>
-        </link>
+        </link> -->
     </xacro:macro>
 </robot>

File: src/arm_robot/description/arm_description.urdf.xacro (robot description, xacro)
@@ -6,13 +6,13 @@
         <xacro:property name="mass" value="1" /> <!-- arbitrary value for mass -->
         <xacro:property name="width" value="0.1" /> <!-- Square dimensions (widthxwidth) of beams -->
-        <xacro:property name="height1" value="2" /> <!-- Link 1 -->
+        <xacro:property name="height1" value="1" /> <!-- Link 1 -->
         <xacro:property name="height2" value="1" /> <!-- Link 2 -->
         <xacro:property name="offset" value="0.05" />
-        <joint name="${prefix}base" type="fixed">
-            <xacro:insert_block name="origin" />
-            <parent link="${parent}" />
-            <child link="${prefix}arm1"/>
+        <joint name="${prefix}base_joint" type="fixed">
+            <xacro:insert_block name="origin"/>
+            <parent link="${parent}"/>
+            <child link="${prefix}base_link"/>
         </joint>
-        <link name="${prefix}arm1">
+        <link name="${prefix}base_link">
             <collision>
                 <origin xyz="0 0 ${height1 / 2}" rpy="0 0 0"/>
@@ -28,5 +28,5 @@
             </visual>
             <interial>
-                <origin xyz="0 0 ${height1 / 2}"/>
+                <origin xyz="0 0 ${height1 / 2}" rpy="0 0 0"/>
                 <mass value="${mass}" />
                 <inertia ixx="${mass / 12 * (width*width + height1*height1)}" ixy="0.0" ixz="0.0" iyy="{mass / 12 * (width*width + height1*height1)}" iyz="0.0" izz="{mass / 12 * 2*width*width}"/>
@@ -34,14 +34,14 @@
         </link>
         <joint name="${prefix}joint1" type="revolute">
-            <parent link="${prefix}arm1"/>
-            <child link="${prefix}arm2"/>
-            <origin xyz="0 ${width} ${height1 / 2 - offset}"/>
+            <parent link="${prefix}base_link"/>
+            <child link="${prefix}arm1_link"/>
+            <origin xyz="0 ${width} ${height1 - offset}" rpy="0 0 0"/>
             <axis xyz="0.0 1.0 0.0"/>
             <limit lower="${-pi}" upper="${pi}" effort="10" velocity="10"/>
             <dynamics damping="0.7"/>
         </joint>
-        <link name="${prefix}arm2">
+        <link name="${prefix}arm1_link">
             <collision>
-                <origin xyz="0 ${width} ${height2 / 2 - offset}" rpy="0 0 0"/>
+                <origin xyz="0 0 ${height2 / 2}" rpy="0 0 0"/>
                 <geometry>
                     <box size="${width} ${width} ${height2}"/>
@@ -49,5 +49,5 @@
             </collision>
             <visual>
-                <origin xyz="0 ${width} ${height2 / 2 - offset}" rpy="0 ${pi} 0"/>
+                <origin xyz="0 0 ${height2 / 2}" rpy="0 0 0"/>
                 <geometry>
                     <box size="${width} ${width} ${height2}"/>
@@ -55,5 +55,5 @@
             </visual>
             <interial>
-                <origin xyz="0 0 ${height2 / 2 - offset}"/>
+                <origin xyz="0 0 ${height2 / 2}" rpy="0 0 0"/>
                 <mass value="${mass}" />
                 <inertia ixx="${mass / 12 * (width*width + height2*height2)}" ixy="0.0" ixz="0.0" iyy="{mass / 12 * (width*width + height2*height2)}" iyz="0.0" izz="{mass / 12 * 2*width*width}"/>
