Commit message: add arm_sensor

File: install/arm_robot/share/arm_robot/arm_description.urdf.xacro (robot description, xacro)
@@ -49,5 +49,5 @@
             </collision>
             <visual>
-                <origin xyz="0 ${width} ${height2 / 2 -offset}" rpy="0 0 0"/>
+                <origin xyz="0 ${width} ${height2 / 2 - offset}" rpy="0 ${pi} 0"/>
                 <geometry>
                     <box size="${width} ${width} ${height2}"/>
@@ -55,5 +55,5 @@
             </visual>
             <interial>
-                <origin xyz="0 0 ${height2}"/>
+                <origin xyz="0 0 ${height2 / 2 - offset}"/>
                 <mass value="${mass}" />
                 <inertia ixx="${mass / 12 * (width*width + height2*height2)}" ixy="0.0" ixz="0.0" iyy="{mass / 12 * (width*width + height2*height2)}" iyz="0.0" izz="{mass / 12 * 2*width*width}"/>

Commit message: launch file for sensor arm works

File: install/arm_robot/share/arm_robot/arm_description.urdf.xacro (robot description, xacro)
@@ -33,5 +33,5 @@
             </interial>
         </link>
-        <!-- <joint name="${prefix}joint1" type="revolute">
+        <joint name="${prefix}joint1" type="revolute">
             <parent link="${prefix}base_link"/>
             <child link="${prefix}arm1_link"/>
@@ -59,5 +59,5 @@
                 <inertia ixx="${mass / 12 * (width*width + height2*height2)}" ixy="0.0" ixz="0.0" iyy="{mass / 12 * (width*width + height2*height2)}" iyz="0.0" izz="{mass / 12 * 2*width*width}"/>
             </interial>
-        </link> -->
+        </link>
     </xacro:macro>
 </robot>

File: install/arm_robot/share/arm_robot/arm_sensor.urdf.xacro (robot description, xacro)
@@ -4,5 +4,6 @@
     <!-- As we move through the file, new things to note will be pointed out. -->
     <!-- It's not meant an example of GOOD design, but an example of some of the various features of URDF/xacro. -->
-    <xacro:include filename="inertials.urdf.xacro" />
+    <xacro:include filename="inertials.xacro" />
+    <xacro:include filename="materials.xacro" />
     <!-- This first link called "world" is empty -->
     <link name="world"></link>
